File: hardware/c92_decoder.kicad_sch (KiCad schematic)
At the start: 83 parts, among them J1 TRACK_1, J10 F2_OUT, J11 F3_OUT, J12 F4_OUT, J13 GND, J14 CAP, J2 SWD, J3 TRACK_2, J4 F0F_OUT, J5 F0R_OUT, J6 MOTOR_L, J7 MOTOR_R, J8 VDD, J9 F1_OUT, Q1 DMC3071LVT, Q2 DMC3071LVT, Q3 DDC114YU, Q4 DDC114YU, Q5 DMN3190LDW, Q6 DMN3190LDW, Q7 DMN3190LDW, SW1 ADDRESS, U1 TPS70933DBVR, U2 STM32G031G8U6, U3 INA180A3

Commit message: Updated title blocks of PCBA projects
Other:
- company: Slonket -> https://github.com/slonket/c92-decoder
Changed lines of the file:
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@@
 	(title_block
 		(title "c92 decoder")
-		(date "2026-04-12")
+		(date "2026-08-14")
 		(rev "REV-A1")
-		(company "Slonket")
+		(company "https://github.com/slonket/c92-decoder")
 	)
 	(rectangle
