File: tools/discrete_hbridge/discrete_hbridge.kicad_sch (KiCad schematic)
At the start: 58 parts, among them J1 MOTOR, J2 MOTOR_H, J3 L_SEL, J4 R_SEL, J5 GND_SEL, J6 OUTPUT, J7 INPUT, J8 OUT, J9 TRACK, Q1 DMC3071LVT, Q2 DMC3071LVT, Q3 MMBT3904, Q4 MMBT3904, Q5 MMBT3904, Q6 2N7002, U1 INA180A2, U2 TPS70933DBVR

Commit message: Updated title blocks of PCBA projects
Other:
- company: Slonket -> https://github.com/slonket/c92-decoder
Changed lines of the file:
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@@
 	(title_block
 		(title "Decoder H-Bridge Development Board")
-		(date "2026-05-15")
+		(date "2026-08-14")
 		(rev "REV-A1")
-		(company "Slonket")
+		(company "https://github.com/slonket/c92-decoder")
 	)
 	(text "H-BRIDGE"
