File: hardware/c92_decoder_B1/c92_decoder_B1.kicad_pcb (KiCad board)
At the start: 4 copper layers, 49 x 34 mm, 93 parts, among them J1 TRACK_1, J10 F2_OUT, J11 F3_OUT, J12 F4_OUT, J13 GND, J14 CAP, J2 SWD, J3 TRACK_2, J4 F0F_OUT, J5 F0R_OUT, J6 MOTOR_L, J7 MOTOR_R, J8 VDD, J9 F1_OUT, Q1 DMC3071LVT, Q2 DMC3071LVT, Q3 DDC114YU, Q4 DDC114YU, Q5 DMN3190LDW, Q6 DMN3190LDW, Q7 DMN3190LDW, SW1 ADDRESS, U1 TPS70933DBVR, U2 STM32G031G8U6, U3 INA180A3

Commit message: started B1 hardware
Parts:
- removed C10, C12: 100n, Slonket_Footprints:C_0603
- removed C11, C13: 10u, Slonket_Footprints:C_1206
- removed C14, C15, C16: 100n, Slonket_Footprints:C_0402
- removed Q1, Q2: DMC3071LVT, Slonket_Footprints:U_SOT-23-6
- removed Q3: DDC114YU, Slonket_Footprints:U_SOT-363
- removed R10, R11, R17: 47k, Slonket_Footprints:R_0402
- removed R12, R13, R14: 10k, Slonket_Footprints:R_0402
- removed R15: 5k1, Slonket_Footprints:R_0402
- removed R16: 20m, Slonket_Footprints:R_0603
- removed R4, R5, R6, R7, R8, R9: 1k, Slonket_Footprints:R_0402
- removed U3: INA180A3, Slonket_Footprints:U_SOT-23-5
- added C2: 10u, Slonket_Footprints:C_1206, F.Cu at (209.6, 97.5)
- added C2: 10u, Slonket_Footprints:C_1206, F.Cu at (212.0, 97.5)
- added C3: 100n, Slonket_Footprints:C_0603, F.Cu at (210.8, 93.6)
- added C3: 100n, Slonket_Footprints:C_0603, F.Cu at (209.2, 93.5)
- added REF**: U_TI_VQFN-16_3.1x3.1_P0.5_EP1, Slonket_Footprints:U_TI_VQFN-16_3.1x3.1_P0.5_EP1, F.Cu at (206.2, 95.8)
Routing:
- net Net-(Q2A-G): track 14.8 -> 0.00 mm, vias 2 -> 0
- net Net-(Q1A-G): track 9.32 -> 21.3 mm, vias 2 -> 0
- net GND: track 18.5 -> 11.0 mm, vias 35 -> 25
- net Net-(C14-Pad1): track 4.30 -> 0.00 mm
- net /P_COM: track 4.27 -> 0.00 mm
- net Net-(Q2B-G): track 7.58 -> 4.24 mm, vias 2 -> 0
- net Net-(Q1B-G): track 8.69 -> 5.55 mm, vias 2 -> 0
- net /BRIDGE_L: track 17.8 -> 14.7 mm, vias 2 -> 1
- net /B_GND: track 2.59 -> 0.00 mm, vias 4 -> 0
- net VDD: track 4.55 -> 2.65 mm, vias 14 -> 10
- net /MOTOR_R: track 16.5 -> 14.9 mm, vias 2 -> 1
- net /MOTOR_L: track 15.8 -> 14.2 mm, vias 2 -> 1
- net +3V3: track 10.6 -> 9.09 mm, vias 6 -> 5
- net /TRACK_2: track 13.0 -> 11.5 mm
- net /BRIDGE_R: track 16.0 -> 14.8 mm, vias 3 -> 1
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- removed copper zone on F.Cu, net (none)
- removed copper zone on F.Cu, net /B_GND
- removed copper zone on F.Cu, net /P_COM
- removed copper zone on F.Cu, net Net-(C14-Pad1)
- removed copper zone on F.Cu, net Net-(Q1A-G)
- removed copper zone on F.Cu, net Net-(Q1B-G)
- removed copper zone on F.Cu, net Net-(Q2A-G)
- removed copper zone on F.Cu, net Net-(Q2B-G)
- removed copper zone on F.Cu, net Net-(Q3A-C1)
- removed copper zone on F.Cu, net Net-(Q3B-C2)
- removed copper zone on F.Cu, net Net-(R17-Pad1)
