File: hardware/c92_decoder_A2/c92_decoder_A2.kicad_pcb (KiCad board)
At the start: 4 copper layers, 49 x 34 mm, 93 parts, among them J1 TRACK_1, J10 F2_OUT, J11 F3_OUT, J12 F4_OUT, J13 GND, J14 CAP, J2 SWD, J3 TRACK_2, J4 F0F_OUT, J5 F0R_OUT, J6 MOTOR_L, J7 MOTOR_R, J8 VDD, J9 F1_OUT, Q1 DMC3071LVT, Q2 DMC3071LVT, Q3 DDC114YU, Q4 DDC114YU, Q5 DMN3190LDW, Q6 DMN3190LDW, Q7 DMN3190LDW, SW1 ADDRESS, U1 TPS70933DBVR, U2 STM32G031G8U6, U3 INA180A3

Commit message: made c92 core; modular decoder layout
Parts:
- J1: value TRACK_1 -> SWD; footprint Slonket_Footprints:J_Pad_1mm_2mm -> Slonket_Footprints:J_Pad_4_1.5mm; moved to B.Cu
- J2: value SWD -> TRACK_1; footprint Slonket_Footprints:J_Pad_4_1.5mm -> Slonket_Footprints:J_Pad_1mm_2mm; moved to F.Cu
- moved J1 30.1 mm to (231.2, 84.0), turned to 0 degrees
- moved J2 30.1 mm to (201.2, 82.0), turned to -90 degrees
Connections:
- net /ADDR_0 renamed /C92 CORE/ADDR_0
- net /ADDR_1 renamed /C92 CORE/ADDR_1
- net /ADDR_2 renamed /C92 CORE/ADDR_2
- net /ADDR_3 renamed /C92 CORE/ADDR_3
- net /ADDR_4 renamed /C92 CORE/ADDR_4
- net /ADDR_5 renamed /C92 CORE/ADDR_5
- net /ADDR_6 renamed /C92 CORE/ADDR_6
- net /ADDR_7 renamed /C92 CORE/ADDR_7
- net /A_SET renamed /C92 CORE/A_SET
- net /BRIDGE_L renamed /C92 CORE/BRIDGE_L
- net /BRIDGE_R renamed /C92 CORE/BRIDGE_R
- net /B_GND renamed /C92 CORE/B_GND
- net /DATA_RX renamed /C92 CORE/DATA_RX
- net /F0F_GPIO renamed /C92 CORE/F0F_GPIO
- net /F0F_OUT renamed /C92 CORE/F0F_OUT
- net /F0R_GPIO renamed /C92 CORE/F0R_GPIO
- net /F0R_OUT renamed /C92 CORE/F0R_OUT
- net /F1_GPIO renamed /C92 CORE/F1_GPIO
- net /F1_OUT renamed /C92 CORE/F1_OUT
- net /F2_GPIO renamed /C92 CORE/F2_GPIO
- net /F2_OUT renamed /C92 CORE/F2_OUT
- net /F3_GPIO renamed /C92 CORE/F3_GPIO
- net /F3_OUT renamed /C92 CORE/F3_OUT
- net /F4_GPIO renamed /C92 CORE/F4_GPIO
- net /F4_OUT renamed /C92 CORE/F4_OUT
- net /MOTOR_L renamed /C92 CORE/MOTOR_L
- net /MOTOR_R renamed /C92 CORE/MOTOR_R
- net /M_BEMF renamed /C92 CORE/M_BEMF
- net /M_PWM renamed /C92 CORE/M_PWM
- net /NRST renamed /C92 CORE/NRST
- net /P_COM renamed /C92 CORE/P_COM
- net /TRACK_2 renamed /C92 CORE/TRACK_2
- net /V_CAP renamed /C92 CORE/V_CAP
- net /V_PROP_I renamed /C92 CORE/V_PROP_I
- net /V_SET renamed /C92 CORE/V_SET
- net /V_VDD renamed /C92 CORE/V_VDD
- D1 pad 2: /TRACK_1 -> /C92 CORE/TRACK_1
- D3 pad 1: /TRACK_1 -> /C92 CORE/TRACK_1
- J1 pad 1: /TRACK_1 -> +3V3
- J2 pad 1: +3V3 -> /C92 CORE/TRACK_1
- U2 pad 20: /SWDIO -> /C92 CORE/SWDIO
- U2 pad 21: /SWCLK -> /C92 CORE/SWCLK
Routing:
- net /SWCLK: track 18.8 -> 0.00 mm, vias 2 -> 0
- net /C92 CORE/SWCLK: track 0.00 -> 18.8 mm, vias 0 -> 2
- net /SWDIO: track 14.8 -> 0.00 mm, vias 2 -> 0
- net /C92 CORE/SWDIO: track 0.00 -> 14.8 mm, vias 0 -> 2
- added copper zone on B.Cu, net (none)
- added copper zone on B.Cu, net /C92 CORE/SWCLK
- added copper zone on F.Cu, net /C92 CORE/SWCLK
- added copper zone on In1.Cu, net /C92 CORE/SWCLK
- added copper zone on B.Cu, net /C92 CORE/SWDIO
- added copper zone on F.Cu, net /C92 CORE/SWDIO
- added copper zone on In1.Cu, net /C92 CORE/SWDIO
- added copper zone on F.Cu, net /C92 CORE/TRACK_1
- removed copper zone on B.Cu, net /SWCLK
- removed copper zone on F.Cu, net /SWCLK
- removed copper zone on In1.Cu, net /SWCLK
- removed copper zone on B.Cu, net /SWDIO
- removed copper zone on F.Cu, net /SWDIO
- removed copper zone on In1.Cu, net /SWDIO
- removed copper zone on F.Cu, net /TRACK_1
