File: hardware/c92_decoder_A2/c92_decoder_A2.kicad_sch (KiCad schematic)
At the start: 83 parts, among them J1 TRACK_1, J10 F2_OUT, J11 F3_OUT, J12 F4_OUT, J13 GND, J14 CAP, J2 SWD, J3 TRACK_2, J4 F0F_OUT, J5 F0R_OUT, J6 MOTOR_L, J7 MOTOR_R, J8 VDD, J9 F1_OUT, Q1 DMC3071LVT, Q2 DMC3071LVT, Q3 DDC114YU, Q4 DDC114YU, Q5 DMN3190LDW, Q6 DMN3190LDW, Q7 DMN3190LDW, SW1 ADDRESS, U1 TPS70933DBVR, U2 STM32G031G8U6, U3 INA180A3

Commit message: added REV-A2 hardware (BOM change)
Parts:
- C14, R15: now not fitted
Other:
- note removed: "Output is approx 1/4"

Commit message: made c92 core; modular decoder layout
Parts:
- removed C1, C11, C13, C2: 10u, Slonket_Footprints:C_1206, symbol Device:C
- removed C10, C12, C3: 100n, Slonket_Footprints:C_0603, symbol Device:C
- removed C14, C15, C16, C17, C18, C6, C7, C9: 100n, Slonket_Footprints:C_0402, symbol Device:C
- removed C4, C8: 4u7, Slonket_Footprints:C_0402, symbol Device:C
- removed C5: 100u, Slonket_Footprints:CP_1210_CASE_B, symbol Device:C_Polarized
- removed D1, D2, D3, D4, D8: DSK34, Slonket_Footprints:D_SOD-123F, symbol Device:D_Schottky
- removed D5: BZD27C27P, Slonket_Footprints:D_SOD-123F, symbol Device:D_Zener
- removed J2: SWD, Slonket_Footprints:J_Pad_4_1.5mm, symbol Connector_Generic:Conn_01x04
- removed Q1, Q2: DMC3071LVT, Slonket_Footprints:U_SOT-23-6, symbol Transistor_FET:DMC3071LVT
- removed Q3, Q4: DDC114YU, Slonket_Footprints:U_SOT-363, symbol Transistor_BJT:Q_Dual_NPN_NPN_BRT_E1B1C2E2B2C1
- removed Q5, Q6, Q7: DMN3190LDW, Slonket_Footprints:U_SOT-363, symbol Transistor_FET:Q_Dual_NMOS_S1G1D2S2G2D1
- removed R1: 100k, Slonket_Footprints:R_0402, symbol Device:R
- removed R10, R11, R17, R20, R21, R24, R25, R28, R29, R32: 47k, Slonket_Footprints:R_0402, symbol Device:R
- removed R12, R13, R14, R2, R31: 10k, Slonket_Footprints:R_0402, symbol Device:R
- removed R15: 5k1, Slonket_Footprints:R_0402, symbol Device:R
- removed R16: 20m, Slonket_Footprints:R_0603, symbol Device:R
- removed R18, R19, R22, R23, R26, R27, R4, R5, R6, R7, R8, R9: 1k, Slonket_Footprints:R_0402, symbol Device:R
- removed R3: 12k, Slonket_Footprints:R_0402, symbol Device:R
- removed R30: 220, Slonket_Footprints:R_0805, symbol Device:R
- removed RV1, RV2: 3314J-1-104E, Slonket_Footprints:RV_BOURNS_3314J, symbol Device:R_Potentiometer
- removed SW1: ADDRESS, Slonket_Footprints:SW_DIP_8_P1.27, symbol Switch:SW_DIP_x08
- removed U1: TPS70933DBVR, Slonket_Footprints:U_SOT-23-5, symbol Slonket_Symbols:TPS70933DBVR
- removed U2: STM32G031G8U6, Slonket_Footprints:U_STM_UFQFPN-28_4x4_P0.5, symbol Slonket_Symbols:STM32G031G6Ux
- removed U3: INA180A3, Slonket_Footprints:U_SOT-23-5, symbol Amplifier_Current:INA180A2
- renumbered J1 to J2
Connections:
- net F0F_OUT renamed C92 CORE/F0F_OUT
- net F0R_OUT renamed C92 CORE/F0R_OUT
- net F1_OUT renamed C92 CORE/F1_OUT
- net F2_OUT renamed C92 CORE/F2_OUT
- net F3_OUT renamed C92 CORE/F3_OUT
- net F4_OUT renamed C92 CORE/F4_OUT
- net GND renamed C92 CORE/GND
- net MOTOR_L renamed C92 CORE/MOTOR_L
- net MOTOR_R renamed C92 CORE/MOTOR_R
- net TRACK_1 renamed C92 CORE/TRACK_1
- net TRACK_2 renamed C92 CORE/TRACK_2
- net VDD renamed C92 CORE/VDD
- net V_CAP renamed C92 CORE/V_CAP
- no-connect marks 1 -> 0
Other:
- added sheet C92 CORE (c92_core_A2.kicad_sch)
- note removed: "Any 3314J potentiometer can be used. 100k is selected to minimise passive current draw from LDO."
- note removed: "BEMF SENSING"
- note removed: "CONFIGURATION"
- note removed: "CURRENT SENSING"
- note removed: "DUAL NFET CANDIDATES: - DMN3190LDW - V_{DS}=30V, R_{DS}=335m@4.5V, I_D=750mA - LCSC=C154750 - SOT-363 - $0.10 - US6K1TR - V_{DS}=30V, R_{DS}=240m@4.5V, I_D=1.5A - LCSC=C703686 - SOT-363T - $0.13"
- note removed: "FUNCTION DRIVERS"
- note removed: "Gain = 2V/A"
- note removed: "LDO CANDIDATES: - TPS70933DBVR - V_{in}=30V, I_{out}=150mA, C_{out}=2.2uF-47uF - LCSC=C89347 - $0.15 - TPS7B6933DBVR - V_{in}=40V, I_{out}=150mA, C_{out}=2.2uF-100uF - additional GND thermal sink - LCSC=C5371018 - $0.43"
- note removed: "MCU OPTIONS: - STM32G031G6U6 - 32kB/8kB - LCSC: C724053 - $0.90 (10+) - STM32G031G8U6 - 64kB/8kB - LCSC: C432211 - $0.90 (10+) - much higher inventory"
- note removed: "MICROCONTROLLER"
- note removed: "MOTOR DRIVER"
- note removed: "NC connects to GND in layout example (pg.16)"
- note removed: "OPTIONS: - C18198103 - C19189054"
- note removed: "PERIPHERAL ALLOCATION - TIM1 - CH1 -> M_PWM - CH5 -> TRGO2 to ADC for BEMF - BRK <- ~{M_FAULT} - TIM2 (32-bit) - CH1 -> DATA_RX - TIM3 (all channels interchangeable) - CH1 -> F0F - CH2 -> F0R - CH3 -> F3 - CH3 -> F4 - ADC - M_BEMF (TRGO in) - V_SET - A_SET - V_VDD - I_MOTOR"
- note removed: "POWER"
- note removed: "R_{AIN} = 50k MAX"
- note removed: "SIGNAL LEVEL SHIFTER"
- note removed: "WIRING"
- moved on the sheet: J10, J11, J12, J13, J14, J2, J3, J4, J5, J6, J7, J8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
