File: hardware/c92_decoder_A2/c92_core_A2.kicad_sch (KiCad schematic)
At the start: 70 parts, among them J1 SWD, Q1 DMC3071LVT, Q2 DMC3071LVT, Q3 DDC114YU, Q4 DDC114YU, Q5 DMN3190LDW, Q6 DMN3190LDW, Q7 DMN3190LDW, SW1 ADDRESS, U1 TPS70933DBVR, U2 STM32G031G8U6, U3 INA180A3

Commit message: new KiCAD structure for multiple variants
Other:
- title: c92 decoder -> c92 decoder - core
Changed lines of the file:
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@@
 	(paper "A3")
 	(title_block
-		(title "c92 decoder")
+		(title "c92 decoder - core")
 		(date "2026-10-05")
 		(rev "REV-A2")
